Commit message: first trial for grasp gen

File: rendering-test/ycb-urdfs/003_cracker_box_google_16k_textured_scale_1000.urdf (robot description, URDF)
Before this commit: robot 003_cracker_box, 1 links, 0 joints
Links:
- link baseLink: geometry collision mesh filename=../../urdfs/ycb-tools/models/ycb/003_cracker_box/google_16k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 scale=1.0 1.0 1.0; visual mesh filename=../../urdfs/ycb-tools/models/ycb/003_cracker_box/google_16k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 scale=1.0 1.0 1.0

File: rendering-test/ycb-urdfs/005_tomato_soup_can_google_16k_textured_scale_1000.urdf (robot description, URDF)
Before this commit: robot 005_tomato_soup_can, 1 links, 0 joints
Links:
- link baseLink: geometry collision mesh filename=../../urdfs/ycb-tools/models/ycb/005_tomato_soup_can/google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 scale=1.0 1.0 1.0; visual mesh filename=../../urdfs/ycb-tools/models/ycb/005_tomato_soup_can/google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 scale=1.0 1.0 1.0

File: rendering-test/ycb-urdfs/006_mustard_bottle_google_16k_textured_scale_1000.urdf (robot description, URDF)
Before this commit: robot 006_mustard_bottle, 1 links, 0 joints
Links:
- link baseLink: geometry collision mesh filename=../../urdfs/ycb-tools/models/ycb/006_mustard_bottle/google_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 scale=1.0 1.0 1.0; visual mesh filename=../../urdfs/ycb-tools/models/ycb/006_mustard_bottle/google_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 scale=1.0 1.0 1.0

File: rendering-test/ycb-urdfs/007_tuna_fish_can_google_16k_textured_scale_1000.urdf (robot description, URDF)
Before this commit: robot 007_tuna_fish_can, 1 links, 0 joints
Links:
- link baseLink: geometry collision mesh filename=/root/data/urdfs/ycb-tools/models/ycb/007_tuna_fish_can/goo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 scale=1.0 1.0 1.0; visual mesh filename=/root/data/urdfs/ycb-tools/models/ycb/007_tuna_fish_can/goo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 scale=1.0 1.0 1.0

File: rendering-test/ycb-urdfs/008_pudding_box_google_16k_textured_scale_1000.urdf (robot description, URDF)
Before this commit: robot 008_pudding_box, 1 links, 0 joints
Links:
- link baseLink: geometry collision mesh filename=/root/data/urdfs/ycb-tools/models/ycb/008_pudding_box/googl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 scale=1.0 1.0 1.0; visual mesh filename=/root/data/urdfs/ycb-tools/models/ycb/008_pudding_box/googl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 scale=1.0 1.0 1.0

File: rendering-test/ycb-urdfs/009_gelatin_box_google_16k_textured_scale_1000.urdf (robot description, URDF)
Before this commit: robot 009_gelatin_box, 1 links, 0 joints
Links:
- link baseLink: geometry collision mesh filename=/root/data/urdfs/ycb-tools/models/ycb/009_gelatin_box/googl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 scale=1.0 1.0 1.0; visual mesh filename=/root/data/urdfs/ycb-tools/models/ycb/009_gelatin_box/googl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 scale=1.0 1.0 1.0

File: rendering-test/ycb-urdfs/010_potted_meat_can_google_16k_textured_scale_1000.urdf (robot description, URDF)
Before this commit: robot 010_potted_meat_can, 1 links, 0 joints
Links:
- link baseLink: geometry collision mesh filename=/root/data/urdfs/ycb-tools/models/ycb/010_potted_meat_can/g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 scale=1.0 1.0 1.0; visual mesh filename=/root/data/urdfs/ycb-tools/models/ycb/010_potted_meat_can/g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 scale=1.0 1.0 1.0

File: rendering-test/ycb-urdfs/021_bleach_cleanser_google_16k_textured_scale_1000.urdf (robot description, URDF)
Before this commit: robot 021_bleach_cleanser, 1 links, 0 joints
Links:
- link baseLink: geometry collision mesh filename=/root/data/urdfs/ycb-tools/models/ycb/021_bleach_cleanser/g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 scale=1.0 1.0 1.0; visual mesh filename=/root/data/urdfs/ycb-tools/models/ycb/021_bleach_cleanser/g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 scale=1.0 1.0 1.0
